File: Wifi_Shielf_KiCad_Files/_autosave-OpenBCI_Wifi_Shield.sch (KiCad schematic (older format))
At the start: 35 parts, among them P1 CONN_01X04, P10 CONN_01X04, P2 CONN_01X04, P4 CONN_01X02, P5 CONN_01X02, P6 CONN_01X02, P7 CONN_01X08, P8 CONN_01X08, P9 CONN_01X04, SW1 TACT_SWITCH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

Commit message: Adição dos gerber files e layout da pcb
Parts:
- J1, J2: renamed from J?; footprint (none) -> Connector_PinHeader_2.54mm:PinHeader_1x05_P2.54mm_Vertical
- gave numbers to parts that had none: 2
Connections:
- net 9V is gone; now on net 6V: IC1.4 (MIRROR_OUTPUT), IC1.7 (I2_HIGH), IC1.8 (I1_HIGH), IC2.14 (VDD)
- net 6V: now reaches R2.1, SW3.1 (T), U2.1 (IN)
Changed lines of the file:
@@
 $EndComp
 Wire Wire Line
-	6850 2300 7200 2300
+	6850 2300 7050 2300
 Wire Wire Line
 	8200 3550 8550 3550
@@
 	5150 5000 5250 5000
 $Comp
-L REF200AU:REF200AU IC?
+L REF200AU:REF200AU IC1
 U 1 1 6316B43A
 P 6100 7700
-F 0 "IC?" H 7100 7965 50  0000 C CNN
+F 0 "IC1" H 7100 7965 50  0000 C CNN
 F 1 "REF200AU" H 7100 7874 50  0000 C CNN
 F 2 "SOIC127P600X175-8N" H 7950 7800 50  0001 L CNN
@@
 $EndComp
 $Comp
-L CD4066BE:CD4066BE IC?
+L CD4066BE:CD4066BE IC2
 U 1 1 6316C4E8
 P 6200 8650
-F 0 "IC?" H 7150 8915 50  0000 C CNN
+F 0 "IC2" H 7150 8915 50  0000 C CNN
 F 1 "CD4066BE" H 7150 8824 50  0000 C CNN
 F 2 "DIP794W53P254L1930H508Q14N" H 7950 8750 50  0001 L CNN
@@
 COMM
 Text Label 6000 8000 2    60   ~ 0
-9V
+6V
 Text Label 8150 7500 0    60   ~ 0
-9V
+6V
 Wire Wire Line
 	8100 7800 8150 7800
@@
 C_C
 $Comp
-L power:GND #PWR?
+L power:GND #PWR024
 U 1 1 631942E9
 P 6050 9350
-F 0 "#PWR?" H 6050 9100 50  0001 C CNN
+F 0 "#PWR024" H 6050 9100 50  0001 C CNN
 F 1 "GND" H 6050 9200 50  0000 C CNN
 F 2 "" H 6050 9350 50  0000 C CNN
@@
 	6050 8650 6200 8650
 Text Label 8250 8650 0    60   ~ 0
-9V
+6V
 Wire Wire Line
 	8100 8650 8250 8650
@@
 C_C
 $Comp
-L Connector:Conn_01x05_Female J?
+L Connector:Conn_01x05_Female J2
 U 1 1 631EBAD7
 P 4700 9150
-F 0 "J?" H 4592 8725 50  0000 C CNN
+F 0 "J2" H 4592 8725 50  0000 C CNN
 F 1 "Conn_4x1_HDTDCS_Cathode(-)" H 4750 8800 50  0000 C CNN
-F 2 "" H 4700 9150 50  0001 C CNN
+F 2 "Connector_PinHeader_2.54mm:PinHeader_1x05_P2.54mm_Vertical" H 4700 9150 50  0001 C CNN
 F 3 "~" H 4700 9150 50  0001 C CNN
 	1    4700 9150
@@
 $EndComp
 $Comp
-L power:GND #PWR?
+L power:GND #PWR023
 U 1 1 6317ABCD
 P 5100 9500
-F 0 "#PWR?" H 5100 9250 50  0001 C CNN
+F 0 "#PWR023" H 5100 9250 50  0001 C CNN
 F 1 "GND" H 5100 9350 50  0000 C CNN
 F 2 "" H 5100 9500 50  0000 C CNN
@@
 	4900 8950 5150 8950
 $Comp
-L Connector:Conn_01x05_Female J?
+L Connector:Conn_01x05_Female J1
 U 1 1 632256B4
 P 4500 8050
-F 0 "J?" H 4300 7600 50  0000 C CNN
+F 0 "J1" H 4300 7600 50  0000 C CNN
 F 1 "Conn_4x1_HDTDCS_Anode(+)" H 4300 7700 50  0000 C CNN
-F 2 "" H 4500 8050 50  0001 C CNN
+F 2 "Connector_PinHeader_2.54mm:PinHeader_1x05_P2.54mm_Vertical" H 4500 8050 50  0001 C CNN
 F 3 "~" H 4500 8050 50  0001 C CNN
 	1    4500 8050
@@
 $EndComp
 $Comp
-L power:GND #PWR?
+L power:GND #PWR022
 U 1 1 632256BA
 P 5100 7800
-F 0 "#PWR?" H 5100 7550 50  0001 C CNN
+F 0 "#PWR022" H 5100 7550 50  0001 C CNN
 F 1 "GND" H 5100 7650 50  0000 C CNN
 F 2 "" H 5100 7800 50  0000 C CNN
@@
 Wire Wire Line
 	4950 7750 4950 7850
+Text Label 7050 2100 0    60   ~ 0
+6V
+Wire Wire Line
+	7050 2100 7050 2300
+Connection ~ 7050 2300
+Wire Wire Line
+	7050 2300 7200 2300
 $EndSCHEMATC
